File: FTCMS_V2.2/FTCMS_V2.2.kicad_sch (KiCad schematic)
At the start: 113 parts, among them J1 Conn_01x20_Female, J2 Conn_02x10_Odd_Even, J3 ToSlave, J4 ToMaster, J5 Conn_02x02_Odd_Even, Q1 Q_NPN_BCE DZT5551, U1 MAX9031AU, U2 ADBMS1818ASWAZ

Commit message: aufräumen
Parts:
- R25: value R -> 0R
Changed lines of the file:
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@@
       (effects (font (size 1.27 1.27)))
     )
-    (property "Value" "R" (at 229.235 86.36 90)
+    (property "Value" "0R" (at 229.235 86.36 90)
       (effects (font (size 1.27 1.27)))
     )
